File: pcb/mill/Console.sch (KiCad schematic (older format))
At the start: 18 parts, among them J1 CONN_01X26, J2 CONN_01X26

Commit message: PCB update
Parts:
- added J?: Conn_01x03_Female, symbol Connector:Conn_01x03_Female
- added R? (x8): 4R7, symbol Device:R_US
- J3: renamed from J?; value Conn_01x04_Female -> Z_Output; footprint (none) -> Connector_PinHeader_2.54mm:PinHeader_1x04_P2.54mm_Vertical
- J4: renamed from J?; value Conn_01x04_Female -> A_Output
- J5: renamed from J?; value Conn_01x04_Female -> Y_Output; footprint (none) -> Connector_PinHeader_2.54mm:PinHeader_1x04_P2.54mm_Vertical
- J6: renamed from J?; value Conn_01x04_Female -> X_Output; footprint (none) -> Connector_PinHeader_2.54mm:PinHeader_1x04_P2.54mm_Vertical
- gave numbers to parts that had none: 12
- renumbered J2 to J1, J1 to J2
Connections:
- net labels added: A1_Limit, A2_Limit, VCC, X1_Limit, X2_Limit, Y1_Limit, Y2_Limit, Z1_Limit, Z2_Limit
- wire segments 109 -> 128
Other:
- moved on the sheet: J3, J4, J5, J6, R1, R10, R11, R12, R2, R3, R4, R5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
